File: TGD.kicad_pcb (KiCad board)
At the start: 4 copper layers, 64 x 38 mm, 65 parts, among them J100 Conn_01x01_Female, J2 Conn_01x02, J20 FT_switch, J21 Battery High, J22 Battery Low, J23 ESC_VDD, J24 ESC_GND, J3 Conn_01x02, J4 USB_B_Micro, J5 Conn_01x05, J6 Conn_01x06, Q10 AO3401A, Q11 AO3401A, Q12 AO3401A, U1 STM32F030C8Tx, U100 SX1276, U101 Crystal_GND24, U2 Crystal_GND24, U20 SY8253ADC, U30 H3LIS331DL, U40 LE25U40CMD

Commit message: Schematic and Layout first draft completed, need to route next
Parts:
- removed the D10 at (207.0, 140.0)
- removed J100: Conn_01x01_Female, Connector_PinHeader_2.54mm:PinHeader_1x01_P2.54mm_Vertical
- removed J23: ESC_VDD, lib_fp:TGD_ESC_PwrPad2
- removed J24: ESC_GND, lib_fp:TGD_ESC_PwrPad2
- removed L100: 10nH, Inductor_SMD:L_0402_1005Metric
- removed Q10: AO3401A, Package_TO_SOT_SMD:SOT-23
- removed the R10 at (186.7, 138.6)
- removed the R13 at (204.2, 137.5)
- added C111: 8.2pF, Capacitor_SMD:C_0402_1005Metric, F.Cu at (-37.5, 30.9)
- added C112: 1.5pF, Capacitor_SMD:C_0402_1005Metric, F.Cu at (-39.5, 33.0)
- added C113: 3.3pF, Capacitor_SMD:C_0402_1005Metric, F.Cu at (-39.5, 30.9)
- added C117: 3.3pF, Capacitor_SMD:C_0402_1005Metric, F.Cu at (-29.1, 25.1)
- added C118: 47pF, Capacitor_SMD:C_0402_1005Metric, F.Cu at (-31.0, 26.1)
- added C120: 47pF, Capacitor_SMD:C_0402_1005Metric, F.Cu at (-45.3, 34.9)
- added C121: 47pF, Capacitor_SMD:C_0402_1005Metric, F.Cu at (-33.6, 29.9)
- added C122: 1nF, Capacitor_SMD:C_0402_1005Metric, F.Cu at (-43.4, 33.1)
- added C135: 100nF, Capacitor_SMD:C_0402_1005Metric, F.Cu at (-33.6, 28.8)
- added C145: 1nF, Capacitor_SMD:C_0402_1005Metric, F.Cu at (-43.4, 36.5)
- added C7: 2.2uF, Capacitor_SMD:C_0603_1608Metric, F.Cu at (22.9, 23.1)
- added C8: 2.2uF, Capacitor_SMD:C_0603_1608Metric, F.Cu at (15.4, 36.6)
- added D1: B5819W, Diode_SMD:D_SOD-123, F.Cu at (0.25, 34.8)
- added D12: 3V3_LED, LED_SMD:LED_0603_1608Metric_Pad1.05x0.95mm_HandSolder, F.Cu at (-71.0, 52.4)
- added D13: MISC1_LED, LED_SMD:LED_0603_1608Metric_Pad1.05x0.95mm_HandSolder, F.Cu at (-67.6, 50.6)
- added D14: MISC2_LED, LED_SMD:LED_0603_1608Metric_Pad1.05x0.95mm_HandSolder, F.Cu at (-64.2, 48.8)
- added D2: B5819W, Diode_SMD:D_SOD-123, F.Cu at (0.25, 29.5)
- added D50: ZMM3V3, Diode_SMD:D_MiniMELF, F.Cu at (11.3, 1.85)
- added J1: G-Switch-ST-0322, lib_fp:G-Switch-ST-TRRS, B.Cu at (-5.50, 38.3)
- added J103: Conn_01x01_Female, Connector_PinHeader_2.54mm:PinHeader_1x01_P2.54mm_Vertical, F.Cu at (-47.1, 38.0)
- added J104: Conn_01x01_Female, Connector_PinHeader_2.54mm:PinHeader_1x01_P2.54mm_Vertical, F.Cu at (-25.6, 25.0)
- added JP2: SolderJumper_2_Open, lib_fp:TGD_SolderJumper, F.Cu at (16.1, 31.5)
- added JP3: SolderJumper_2_Open, lib_fp:TGD_SolderJumper, F.Cu at (16.1, 30.1)
- added L102: 33nH, Inductor_SMD:L_0402_1005Metric, F.Cu at (-33.7, 30.9)
- added L103: 2.2nH, Inductor_SMD:L_0402_1005Metric, F.Cu at (-33.6, 31.9)
- added L104: 5.6nH, Inductor_SMD:L_0402_1005Metric, F.Cu at (-37.5, 31.9)
- added L105: 4.7nH, Inductor_SMD:L_0402_1005Metric, F.Cu at (-39.5, 31.9)
- added L107: 10nH, Inductor_SMD:L_0402_1005Metric, F.Cu at (-29.1, 26.1)
- added R101: 1K, Resistor_SMD:R_0402_1005Metric, F.Cu at (-43.4, 32.1)
- added R15: 10K, Resistor_SMD:R_0603_1608Metric_Pad0.98x0.95mm_HandSolder, F.Cu at (4.95, 2.45)
- added R16: 1K, Resistor_SMD:R_0603_1608Metric_Pad0.98x0.95mm_HandSolder, F.Cu at (-73.6, 55.6)
- added R17: 1K, Resistor_SMD:R_0603_1608Metric_Pad0.98x0.95mm_HandSolder, F.Cu at (-70.2, 53.8)
- added R18: 1K, Resistor_SMD:R_0603_1608Metric_Pad0.98x0.95mm_HandSolder, F.Cu at (-66.8, 52.0)
- added R19: 1K, Resistor_SMD:R_0603_1608Metric_Pad0.98x0.95mm_HandSolder, F.Cu at (-63.4, 50.2)
- added R2: 22R, Resistor_SMD:R_0603_1608Metric_Pad0.98x0.95mm_HandSolder, F.Cu at (15.6, 34.1)
- added R3: 22R, Resistor_SMD:R_0603_1608Metric_Pad0.98x0.95mm_HandSolder, F.Cu at (15.6, 32.9)
- added U102: PE4259, Package_TO_SOT_SMD:SOT-363_SC-70-6, F.Cu at (-42.9, 34.9)
- added U3: CYCLONE-35A, lib_fp:TGD-ESC-CYCLONE-35A, F.Cu at (-85.0, 42.0)
- added U4: CYCLONE-35A, lib_fp:TGD-ESC-CYCLONE-35A, F.Cu at (85.0, 42.0)
- C108: footprint Capacitor_SMD:C_0402_1005Metric -> Capacitor_SMD:C_0603_1608Metric
- C109: value 47pF -> 22pF
- C110: value 3.3pF -> 8.2pF
- D11: value DOWN_LED -> POWER_LED; footprint LED_THT:LED_D3.0mm -> LED_SMD:LED_0603_1608Metric_Pad1.05x0.95mm_HandSolder
- J2: value Conn_01x02 -> G-Switch-ST-0322; footprint lib_fp:TGD_ESC_SigPads -> lib_fp:G-Switch-ST-TRRS; moved to B.Cu
- J3: value Conn_01x02 -> Conn_01x01; footprint lib_fp:TGD_ESC_SigPads -> lib_fp:TGD_ESC_SigPad
- J4: value USB_B_Micro -> Conn_01x01; footprint lib_fp:USB_Micro-B_uxcell -> lib_fp:TGD_ESC_SigPad
- J5: value Conn_01x05 -> Conn_01x12; footprint Connector_PinSocket_2.54mm:PinSocket_1x05_P2.54mm_Vertical -> Connector_PinHeader_2.54mm:PinHeader_1x12_P2.54mm_Vertical
- J6: value Conn_01x06 -> Conn_01x01; footprint Connector_PinSocket_2.54mm:PinSocket_1x06_P2.54mm_Vertical -> lib_fp:TGD_ESC_PwrPad
- R14: value 33R -> 10K
- U1: value STM32F030C8Tx -> STM32F405RGTx; footprint Package_QFP:LQFP-48_7x7mm_P0.5mm -> Package_QFP:LQFP-64_10x10mm_P0.5mm
- moved J3 296.6 mm to (-62.0, 43.0), turned to 118.25 degrees
- moved D11 267.6 mm to (-74.4, 54.2), turned to -151.75 degrees
- moved R10 241.2 mm to (-4.95, 5.65)
- moved D10 238.5 mm to (2.50, 1.60)
- moved Q11 238.5 mm to (-2.60, 4.05)
- moved Q12 238.5 mm to (2.50, 4.05)
- moved R13 238.5 mm to (0.70, 6.65)
- moved R12 238.4 mm to (-0.60, 6.70)
- moved R11 237.0 mm to (4.95, 5.65)
- moved C109 235.9 mm to (-35.6, 31.9)
- moved J6 235.7 mm to (6.50, 21.5), turned to 0 degrees
- moved U30 234.9 mm to (-15.0, 35.0)
- moved C110 234.9 mm to (-35.6, 30.9), turned to 180 degrees
- moved C22 234.9 mm to (-16.6, 2.46), turned to 90 degrees
- moved C31 234.1 mm to (-15.0, 30.6), turned to 0 degrees
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- renumbered D12 to D10, R11 to R10, R12 to R11, R15 to R12, R16 to R13
Connections:
- C109 pad 1: /sx1276/Antenna -> RFO_HF
- C110 pad 1: Net-(C109-Pad2) -> RFO_HF
- J2 pad 1: GND -> Net-(D2-Pad2)
- J2 pad 2: F_PPM -> Net-(J2-Pad2)
- J20 pad 2: Net-(J20-Pad2) -> VDD
- J21 pad 1: Net-(J20-Pad2) -> GND
- J21 pad 2: VDD -> Net-(J22-Pad1)
- J22 pad 1: GND -> Net-(J22-Pad1)
- J3 pad 1: GND -> PPM_F
- J4 pad 1: +3V3 -> PPM_B
- J5 pad 1: +3V3 -> SNS_VIN
- J5 pad 2: L_INT -> INT_L
- J5 pad 3: B_PPM -> CS_L
- J5 pad 4: F_PPM -> CS_A
- J5 pad 5: GND -> CS_M
- J6 pad 1: P_SCK -> /PGND
- R10 pad 1: BLUE_LED -> LED_BLUE
- R11 pad 1: RED_LED -> LED_RED
- R14 pad 1: Net-(Q10-Pad3) -> +3V3
- R14 pad 2: Net-(D11-Pad2) -> Net-(Q11-Pad1)
- U1 pad 10: SNS_VIN -> unconnected-(U1-Pad10)
- U1 pad 11: Net-(U1-Pad11) -> unconnected-(U1-Pad11)
- U1 pad 12: Net-(U1-Pad12) -> GND
- U1 pad 13: Net-(U1-Pad13) -> +3V3
- U1 pad 14: Net-(U1-Pad14) -> SNS_VIN
- U1 pad 15: P_SCK -> unconnected-(U1-Pad15)
- U1 pad 16: P_MISO -> unconnected-(U1-Pad16)
- U1 pad 17: P_MOSI -> unconnected-(U1-Pad17)
- U1 pad 18: M_CS -> GND
- U1 pad 19: A_CS -> +3V3
- U1 pad 2: Net-(U1-Pad2) -> unconnected-(U1-Pad2)
- U1 pad 20: L_CS -> unconnected-(U1-Pad20)
- U1 pad 21: RED_LED -> P_SCK
- U1 pad 22: DOWN_LED -> P_MISO
- U1 pad 23: GND -> P_MOSI
- U1 pad 24: +3V3 -> unconnected-(U1-Pad24)
- U1 pad 25: BLUE_LED -> unconnected-(U1-Pad25)
- U1 pad 26: STRIP_LED -> CS_M
- U1 pad 27: Net-(U1-Pad27) -> CS_A
- U1 pad 28: Net-(U1-Pad28) -> CS_L
- U1 pad 29: Net-(U1-Pad29) -> LED_BLUE
- U1 pad 3: Net-(U1-Pad3) -> unconnected-(U1-Pad3)
- U1 pad 30: Net-(U1-Pad30) -> LED_RED
- U1 pad 32: Net-(U1-Pad32) -> +3V3
- U1 pad 33: Net-(U1-Pad33) -> LED_MISC1
- U1 pad 34: SWD_DIO -> LED_MISC2
- U1 pad 35: Net-(U1-Pad35) -> unconnected-(U1-Pad35)
- U1 pad 36: Net-(U1-Pad36) -> unconnected-(U1-Pad36)
- U1 pad 37: SWD_CLK -> unconnected-(U1-Pad37)
- U1 pad 38: Net-(U1-Pad38) -> unconnected-(U1-Pad38)
- U1 pad 39: L_INT -> unconnected-(U1-Pad39)
- U1 pad 4: Net-(U1-Pad4) -> unconnected-(U1-Pad4)
- U1 pad 40: Net-(U1-Pad40) -> GPIO_MISC1
- U1 pad 41: Net-(U1-Pad41) -> unconnected-(U1-Pad41)
- U1 pad 42: Net-(U1-Pad42) -> USB_TX
- U1 pad 43: B_PPM -> USB_RX
- U1 pad 44: Net-(R1-Pad2) -> USB_DM
- U1 pad 45: F_PPM -> USB_DP
- U1 pad 46: Net-(U1-Pad46) -> SWD_DIO
- U1 pad 47: GND -> Net-(C8-Pad1)
- U1 pad 8: GND -> unconnected-(U1-Pad8)
- U1 pad 9: +3V3 -> unconnected-(U1-Pad9)
- U100 pad 1: Net-(U100-Pad1) -> unconnected-(U100-Pad1)
- U100 pad 19: L_CS -> CS_L
- U100 pad 20: Net-(U100-Pad20) -> RF_MOD
- U100 pad 21: Net-(L100-Pad1) -> RFI_HF
- U100 pad 22: Net-(U100-Pad22) -> RFO_HF
- U100 pad 25: Net-(U100-Pad25) -> VR_PA
- U100 pad 27: Net-(U100-Pad27) -> PA_BOOST
- U100 pad 28: Net-(U100-Pad28) -> unconnected-(U100-Pad28)
- U100 pad 8: L_INT -> INT_L
- U30 pad 11: Net-(U30-Pad11) -> unconnected-(U30-Pad11)
- U30 pad 2: Net-(U30-Pad2) -> unconnected-(U30-Pad2)
- U30 pad 3: Net-(U30-Pad3) -> unconnected-(U30-Pad3)
- U30 pad 8: A_CS -> CS_A
- U30 pad 9: Net-(U30-Pad9) -> unconnected-(U30-Pad9)
- U40 pad 1: M_CS -> CS_M
Routing:
- net L_INT: track 105.9 -> 0.00 mm, vias 3 -> 0
- net B_PPM: track 82.8 -> 0.00 mm, vias 2 -> 0
- net F_PPM: track 80.6 -> 0.00 mm, vias 2 -> 0
- net P_MISO: track 73.9 -> 0.00 mm, vias 4 -> 0
- net P_MOSI: track 73.7 -> 0.00 mm, vias 3 -> 0
- net P_SCK: track 70.0 -> 0.00 mm, vias 3 -> 0
- net L_CS: track 60.4 -> 0.00 mm, vias 1 -> 0
- net SNS_VIN: track 50.2 -> 3.30 mm, vias 2 -> 1
- net VDD: track 45.8 -> 0.02 mm
- net GND: track 61.3 -> 18.1 mm, vias 35 -> 17
- net DOWN_LED: track 41.6 -> 0.00 mm, vias 2 -> 0
- net +3V3: track 44.4 -> 8.94 mm, vias 18 -> 3
- net SWD_CLK: track 31.4 -> 0.00 mm, vias 2 -> 0
- net M_CS: track 31.1 -> 0.00 mm, vias 1 -> 0
- net A_CS: track 31.0 -> 0.00 mm, vias 1 -> 0
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- removed copper zone on F.Cu, net GND
Other:
- board size 64 x 38 mm -> 175 x 58.5 mm
- net class Default removed
- board text added: "CSA"
- board text added: "CSL"
- board text added: "CSM"
- board text added: "IO1"
- board text added: "IO2"
- board text added: "MO1"
- board text added: "MO2"
- board text added: "PPM_B"
- board text added: "PPM_F"
- board text added: "SPIN-TGD V2"
- board text added: "SVN"
- board text added: "© Jacob Williams 2022"
- board text removed: "ACS"
- board text removed: "BPM"
- board text removed: "FPM"
- board text removed: "LCS"
- board text removed: "MCS"
- board text removed: "TGD V1.0.0"
- board text removed: "© Jacob Williams 2021"

Commit message: last V2 version before switching to separate power and control boards
Parts:
- removed D11: POWER_LED, LED_SMD:LED_0603_1608Metric_Pad1.05x0.95mm_HandSolder
- removed D14: MISC2_LED, LED_SMD:LED_0603_1608Metric_Pad1.05x0.95mm_HandSolder
- removed R16, R19: 1K, Resistor_SMD:R_0603_1608Metric_Pad0.98x0.95mm_HandSolder
- J5: value Conn_01x12 -> Conn_01x06; footprint Connector_PinHeader_2.54mm:PinHeader_1x12_P2.54mm_Vertical -> Connector_PinHeader_2.54mm:PinHeader_1x06_P2.54mm_Vertical
- U100: footprint Package_DFN_QFN:QFN-28-1EP_6x6mm_P0.65mm_EP4.8x4.8mm -> lib_fp:TGD-QFN-28-1EP_6x6mm_P0.65mm_EP4.8x4.8mm
- U30: footprint lib_fp:TFLGA-16_3x3mm -> lib_fp:TGD-TFLGA-16_3x3mm
- moved R14 31.6 mm to (14.7, 27.3), turned to 180 degrees
- moved R10 30.2 mm to (14.7, 28.6), turned to 180 degrees
- moved R15 25.5 mm to (14.7, 26.1), turned to 180 degrees
- moved R11 21.5 mm to (14.7, 24.8), turned to 180 degrees
- moved J104 12.5 mm to (-37.8, 28.2), turned to 45 degrees
- moved Q11 9.61 mm to (6.85, 2.30), turned to 180 degrees
- moved Q12 4.65 mm to (6.85, 5.70), turned to 180 degrees
- moved R12 4.19 mm to (0.00, 2.55)
- moved C50 3.85 mm to (15.1, 4.75)
- moved R50 3.85 mm to (15.1, 6.15)
- moved R51 3.85 mm to (15.1, 3.35)
- moved D10 3.51 mm to (0.00, 4.06)
- moved D50 2.78 mm to (14.1, 1.70)
- moved R13 1.22 mm to (0.00, 5.65)
- moved J5 0.82 mm to (74.0, 55.1)
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Connections:
- net LED_MISC1 renamed LED_MISC
- C145 pad 2: VDD -> +3V3
- J20 pad 1: Net-(J20-Pad1) -> unconnected-(J20-Pad1)
- J21 pad 2: Net-(J22-Pad1) -> unconnected-(J21-Pad2)
- J22 pad 1: Net-(J22-Pad1) -> unconnected-(J22-Pad1)
- J22 pad 2: Net-(J20-Pad1) -> unconnected-(J22-Pad2)
- J5 pad 1: SNS_VIN -> GND
- J5 pad 2: INT_L -> +3V3
- J5 pad 3: CS_L -> P_MISO
- J5 pad 4: CS_A -> P_SCK
- J5 pad 5: CS_M -> P_MOSI
- J5 pad 6: P_MOSI -> GPIO1
- U1 pad 34: LED_MISC2 -> unconnected-(U1-Pad34)
- U1 pad 40: GPIO_MISC1 -> unconnected-(U1-Pad40)
- U1 pad 51: GPIO_MISC2 -> unconnected-(U1-Pad51)
- U1 pad 62: unconnected-(U1-Pad62) -> GPIO1
- U102 pad 6: VDD -> +3V3
- U3 pad 1: VDD -> unconnected-(U3-Pad1)
- U3 pad 2: /PGND -> unconnected-(U3-Pad2)
- U4 pad 1: VDD -> unconnected-(U4-Pad1)
- U4 pad 2: /PGND -> unconnected-(U4-Pad2)
Routing:
- net P_MISO: track 0.00 -> 128.1 mm, vias 0 -> 4
- net P_SCK: track 0.00 -> 124.6 mm, vias 0 -> 4
- net P_MOSI: track 0.00 -> 124.2 mm, vias 0 -> 4
- net LED_MISC: track 0.00 -> 104.8 mm, vias 0 -> 2
- net PPM_F: track 0.00 -> 91.6 mm, vias 0 -> 2
- net +3V3: track 8.94 -> 84.3 mm, vias 3 -> 15
- net CS_L: track 0.00 -> 68.7 mm, vias 0 -> 2
- net VDD: track 0.02 -> 66.0 mm
- net GND: track 18.1 -> 82.8 mm, vias 17 -> 58
- net INT_L: track 0.05 -> 57.1 mm
- net SNS_VIN: track 3.30 -> 49.8 mm, vias 1 -> 2
- net CS_A: track 0.00 -> 44.0 mm, vias 0 -> 2
- net SWD_CLK: track 0.00 -> 42.5 mm, vias 0 -> 1
- net GPIO1: track 0.00 -> 39.0 mm, vias 0 -> 1
- net PPM_B: track 0.00 -> 36.6 mm, vias 0 -> 2
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- added copper zone on F.Cu, net GND
Other:
- outline, holes or cut-outs redrawn
- board text added: "MOL"
- board text removed: "CSA"
- board text removed: "CSL"
- board text removed: "CSM"
- board text removed: "IO1"
- board text removed: "IO2"
- board text removed: "LIT"
- board text removed: "MO1"
- board text removed: "MO2"
- board text removed: "SVN"
- board text removed: "VDD"
