File: TGD.kicad_sch (KiCad schematic)
At the start: 63 parts, among them J1 G-Switch-ST-0322, J2 G-Switch-ST-0322, J20 FT_switch, J21 Battery High, J22 Battery Low, J3 Conn_01x01, J4 Conn_01x01, J5 Conn_01x12, J6 Conn_01x01, Q11 AO3401A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

Commit message: last V2 version before switching to separate power and control boards
Parts:
- removed D11: POWER_LED, LED_SMD:LED_0603_1608Metric_Pad1.05x0.95mm_HandSolder, symbol Device:LED
- removed D14: MISC2_LED, LED_SMD:LED_0603_1608Metric_Pad1.05x0.95mm_HandSolder, symbol Device:LED
- removed J5: Conn_01x12, Connector_PinHeader_2.54mm:PinHeader_1x12_P2.54mm_Vertical, symbol Connector_Generic:Conn_01x12
- removed R16, R19: 1K, Resistor_SMD:R_0603_1608Metric_Pad0.98x0.95mm_HandSolder, symbol Device:R
- added J5: Conn_01x06, Connector_PinHeader_2.54mm:PinHeader_1x06_P2.54mm_Vertical, symbol Connector_Generic:Conn_01x06
- D12, D13: LCSC ! -> (none)
- U30: footprint lib_fp:TFLGA-16_3x3mm -> lib_fp:TGD-TFLGA-16_3x3mm
Connections:
- net +3V3: now also J5.2 (Pin_2)
- net GND: now also J5.1 (Pin_1)
- net PGND: no longer U3.2 (GND), U4.2 (GND)
- net P_MISO: now also J5.3 (Pin_3)
- net P_MOSI: now also J5.5 (Pin_5)
- net P_SCK: now also J5.4 (Pin_4)
- net VDD: no longer U3.1 (VIN), U4.1 (VIN)
- net at J22.1 (Pin_1): no longer J21.2 (Pin_2)
- net at J22.2 (Pin_2): no longer J20.1 (Pin_1)
- net GPIO1: now reaches U1.62 (PB9)
- net GPIO1: now also J5.6 (Pin_6)
- net GPIO_MISC1: no longer names the net of U1.40 (PC9)
- net GPIO_MISC2: no longer names the net of U1.51 (PC10)
- net LED_MISC1 renamed LED_MISC
- net LED_MISC2: no longer names the net of U1.34 (PB13)
