File: sx1276.kicad_sch (KiCad schematic)
At the start: 33 parts, among them J103 Conn_01x01_Female, J104 Conn_01x01_Female, U100 SX1276, U101 Crystal_GND24, U102 PE4259

Commit message: last V2 version before switching to separate power and control boards
Parts:
- C108: LCSC C1525 -> C14663
- U100: footprint Package_DFN_QFN:QFN-28-1EP_6x6mm_P0.65mm_EP4.8x4.8mm -> lib_fp:TGD-QFN-28-1EP_6x6mm_P0.65mm_EP4.8x4.8mm
Connections:
- net VDD is gone; now on net +3V3: C145.2, U102.6 (VDD)
Changed lines of the file:
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@@
   (junction (at 201.93 62.23) (diameter 0) (color 0 0 0 0)
   )
+  (junction (at 72.39 128.27) (diameter 0) (color 0 0 0 0)
+  )
   (junction (at 66.04 48.26) (diameter 0) (color 0 0 0 0)
-  )
-  (junction (at 72.39 128.27) (diameter 0) (color 0 0 0 0)
   )
   (junction (at 72.39 161.29) (diameter 0) (color 0 0 0 0)
@@
     (pin "1")
   )
-  (symbol (lib_id "power:VDD") (at 72.39 128.27 0) (unit 1)
-    (in_bom yes) (on_board yes)
-    (property "Reference" "#PWR0158" (id 0) (at 72.39 132.08 0)
-      (effects (font (size 1.27 1.27)) hide)
-    )
-    (property "Value" "VDD" (id 1) (at 72.771 123.8758 0))
-    (property "Footprint" "" (id 2) (at 72.39 128.27 0)
-      (effects (font (size 1.27 1.27)) hide)
-    )
-    (property "Datasheet" "" (id 3) (at 72.39 128.27 0)
-      (effects (font (size 1.27 1.27)) hide)
-    )
-    (pin "1")
-  )
   (symbol (lib_id "Device:C") (at 212.09 62.23 90) (unit 1)
     (in_bom yes) (on_board yes)
@@
     (property "Reference" "U100" (id 0) (at 123.19 49.53 0))
     (property "Value" "SX1276" (id 1) (at 124.46 46.99 0))
-    (property "Footprint" "Package_DFN_QFN:QFN-28-1EP_6x6mm_P0.65mm_EP4.8x4.8mm" (id 2) (at 101.6 78.74 0)
+    (property "Footprint" "lib_fp:TGD-QFN-28-1EP_6x6mm_P0.65mm_EP4.8x4.8mm" (id 2) (at 101.6 78.74 0)
       (effects (font (size 1.27 1.27)) hide)
     )
@@
       (effects (font (size 1.27 1.27)) hide)
     )
-    (property "Datasheet" "https://lcsc.com/product-detail/Multilayer-Ceramic-Capacitors-MLCC-SMD-SMT_Samsung-Electro-Mechanics-CL05B104KO5NNNC_C1525.html" (id 3) (at 68.58 90.17 0)
-      (effects (font (size 1.27 1.27)) hide)
-    )
-    (property "LCSC" "C1525" (id 4) (at 68.58 90.17 0)
+    (property "Datasheet" "https://lcsc.com/product-detail/Multilayer-Ceramic-Capacitors-MLCC-SMD-SMT_YAGEO-CC0603KRX7R9BB104_C14663.html" (id 3) (at 68.58 90.17 0)
+      (effects (font (size 1.27 1.27)) hide)
+    )
+    (property "LCSC" "C14663" (id 4) (at 68.58 90.17 0)
       (effects (font (size 1.27 1.27)) hide)
     )
@@
       (effects (font (size 1.27 1.27)) hide)
     )
+    (pin "1")
+  )
+  (symbol (lib_id "power:+3V3") (at 72.39 128.27 0) (unit 1)
+    (in_bom yes) (on_board yes)
+    (property "Reference" "#PWR0115" (id 0) (at 72.39 132.08 0)
+      (effects (font (size 1.27 1.27)) hide)
+    )
+    (property "Value" "+3V3" (id 1) (at 72.771 123.8758 0))
+    (property "Footprint" "" (id 2) (at 72.39 128.27 0)
+      (effects (font (size 1.27 1.27)) hide)
+    )
+    (property "Datasheet" "" (id 3) (at 72.39 128.27 0)
+      (effects (font (size 1.27 1.27)) hide)
+    )
