File: spin-tgd-control/spin-tgd-control.kicad_sch (KiCad schematic)
At the start: 53 parts, among them J1 G-Switch-ST-0322, J2 G-Switch-ST-0322, J4 Conn_01x01, J5 Conn_01x01, J6 Conn_01x01, J7 Conn_01x01, J8 Conn_01x06, Q11 AO3401A, Q12 AO3401A, U1 STM32F405RGTx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

Commit message: Moved to new library system
Other:
- note added: "TODO: smarter pin breakouts (testpoints?) removable current limiting - https://www.powerctc.com/en/node/4564 jumper for radius setting DONE: MCU with FPU fix LEDs removable sx1276 receive for usb debuging, have OTG and TTL->RS232 option 3.5mm audio jack for prog and debug more status LEDs Make TRRS Footprint rename labels (ie. F_PPM -> PPM_F) Improve all footprints"
- note removed: "TODO: smarter pin breakouts fix vsns resitor removable current limiting - https://www.powerctc.com/en/node/4564 DONE: MCU with FPU fix LEDs removable sx1276 receive for usb debuging, have OTG and TTL->RS232 option 3.5mm audio jack for prog and debug more status LEDs Make TRRS Footprint rename labels (ie. F_PPM -> PPM_F) Improve all footprints"
Changed lines of the file:
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@@
     (effects (font (size 1.27 1.27)) (justify left bottom))
   )
-  (text "TODO:\nsmarter pin breakouts\nfix vsns resitor\nremovable current limiting - https://www.powerctc.com/en/node/4564\n\nDONE:\nMCU with FPU\nfix LEDs\nremovable sx1276 receive\nfor usb debuging, have OTG and TTL->RS232 option\n3.5mm audio jack for prog and debug\nmore status LEDs\nMake TRRS Footprint\nrename labels (ie. F_PPM -> PPM_F)\nImprove all footprints\n"
+  (text "TODO:\nsmarter pin breakouts (testpoints?)\nremovable current limiting - https://www.powerctc.com/en/node/4564\njumper for radius setting\n\nDONE:\nMCU with FPU\nfix LEDs\nremovable sx1276 receive\nfor usb debuging, have OTG and TTL->RS232 option\n3.5mm audio jack for prog and debug\nmore status LEDs\nMake TRRS Footprint\nrename labels (ie. F_PPM -> PPM_F)\nImprove all footprints\n"
     (at -73.66 121.92 0)
     (effects (font (size 1.27 1.27)) (justify left bottom))

Commit message: created pdfs for V2 schematics
Other:
- note added: "TODO: smarter pin breakouts (testpoints?) removable current limiting - https://www.powerctc.com/en/node/4564 jumper for radius setting"
- note removed: "TODO: smarter pin breakouts (testpoints?) removable current limiting - https://www.powerctc.com/en/node/4564 jumper for radius setting DONE: MCU with FPU fix LEDs removable sx1276 receive for usb debuging, have OTG and TTL->RS232 option 3.5mm audio jack for prog and debug more status LEDs Make TRRS Footprint rename labels (ie. F_PPM -> PPM_F) Improve all footprints"
- company: (none) -> Team Alfredo
- title: (none) -> spin-tgd-control
- moved on the sheet: C50, D12, D13, D50, J8, R17, R18, R50, R51

Commit message: Eggman V2 ordered gerbers
Other:
- note removed: "TODO: smarter pin breakouts (testpoints?) removable current limiting - https://www.powerctc.com/en/node/4564 jumper for radius setting"
Changed lines of the file:
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@@
-    (effects (font (size 1.27 1.27)) (justify left bottom))
-  )
-  (text "TODO:\nsmarter pin breakouts (testpoints?)\nremovable current limiting - https://www.powerctc.com/en/node/4564\njumper for radius setting\n"
-    (at 24.13 189.865 0)
     (effects (font (size 1.27 1.27)) (justify left bottom))
   )
