File: spin-eggman/spin-eggman.kicad_sch (KiCad schematic)
At the start: 16 parts, among them J1 FT_switch, J2 bat_high, J3 bat_low, J4 Conn_01x05, J5 Conn_01x01, J6 Conn_01x01, J8 ESC_Foo, J9 ESC_Bar, U1 INA185A1

Commit message: file cleanup
Parts:
- R1: LCSC (none) -> C2692059
- R3: LCSC (none) -> C21190
Changed lines of the file:
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@@
+      (effects (font (size 1.27 1.27)) hide)
+    )
+    (property "LCSC" "~" (id 4) (at 189.23 102.87 0)
       (effects (font (size 1.27 1.27)) hide)
     )
@@
     )
     (property "Datasheet" "~" (id 3) (at 161.29 68.58 0)
+      (effects (font (size 1.27 1.27)) hide)
+    )
+    (property "LCSC" "~" (id 4) (at 161.29 68.58 0)
       (effects (font (size 1.27 1.27)) hide)
     )
@@
       (effects (font (size 1.27 1.27)) hide)
     )
+    (property "LCSC" "~" (id 4) (at 91.44 102.87 0)
+      (effects (font (size 1.27 1.27)) hide)
+    )
     (pin "1")
     (pin "2")
@@
       (effects (font (size 1.27 1.27)) hide)
     )
+    (property "LCSC" "~" (id 4) (at 158.75 97.79 0)
+      (effects (font (size 1.27 1.27)) hide)
+    )
     (pin "1")
     (pin "2")
@@
     )
     (property "Datasheet" "~" (id 3) (at 158.75 74.93 0)
+      (effects (font (size 1.27 1.27)) hide)
+    )
+    (property "LCSC" "~" (id 4) (at 158.75 74.93 0)
       (effects (font (size 1.27 1.27)) hide)
     )
@@
       (effects (font (size 1.27 1.27)) hide)
     )
+    (property "LCSC" "~" (id 4) (at 151.13 40.64 0)
+      (effects (font (size 1.27 1.27)) hide)
+    )
     (pin "1")
     (pin "2")
@@
     )
     (property "Datasheet" "~" (id 3) (at 91.44 92.71 0)
+      (effects (font (size 1.27 1.27)) hide)
+    )
+    (property "LCSC" "~" (id 4) (at 91.44 92.71 0)
       (effects (font (size 1.27 1.27)) hide)
     )
@@
       (effects (font (size 1.27 1.27)) hide)
     )
+    (property "LCSC" "~" (id 4) (at 91.44 96.52 0)
+      (effects (font (size 1.27 1.27)) hide)
+    )
     (pin "1")
     (pin "2")
@@
       (effects (font (size 1.27 1.27)) hide)
     )
+    (property "LCSC" "~" (id 4) (at 189.23 92.71 0)
+      (effects (font (size 1.27 1.27)) hide)
+    )
     (pin "1")
     (pin "2")
@@
       (effects (font (size 1.27 1.27)) hide)
     )
-    (property "Datasheet" "" (id 3) (at 107.95 93.98 0)
-      (effects (font (size 1.27 1.27)) hide)
-    )
-    (property "LCSC" "" (id 4) (at 107.95 93.98 0)
+    (property "Datasheet" "https://lcsc.com/product-detail/Chip-span-style-background-color-ff0-Resistor-span-Surface-Mount_UNI-ROYAL-Uniroyal-Elec-0603WAF1001T5E_C21190.html" (id 3) (at 107.95 93.98 0)
+      (effects (font (size 1.27 1.27)) hide)
+    )
+    (property "LCSC" "C21190" (id 4) (at 107.95 93.98 0)
       (effects (font (size 1.27 1.27)) hide)
     )
@@
     )
     (property "Datasheet" "~" (id 3) (at 168.91 97.79 0)
+      (effects (font (size 1.27 1.27)) hide)
+    )
+    (property "LCSC" "~" (id 4) (at 168.91 97.79 0)
       (effects (font (size 1.27 1.27)) hide)
     )
@@
       (effects (font (size 1.27 1.27)) hide)
     )
-    (property "Datasheet" "" (id 3) (at 135.89 105.41 0)
-      (effects (font (size 1.27 1.27)) hide)
-    )
+    (property "Datasheet" "https://lcsc.com/product-detail/Chip-span-style-background-color-ff0-Resistor-span-Surface-Mount_SART-Nanjing-Sart-Tech-SMF25M2F2M50T_C2692059.html" (id 3) (at 135.89 105.41 0)
+      (effects (font (size 1.27 1.27)) hide)
+    )
+    (property "LCSC" "C2692059" (id 4) (at 135.89 105.41 0)
+      (effects (font (size 1.27 1.27)) hide)
+    )

Commit message: added image folder and Spin-Sonic PDF
Other:
- note added: "TODO: startup current limiting - https://www.powerctc.com/en/node/4564 Errata: Flip an ESC upside down to fix topology issue Investigate using traces with vias for high current 10mm 2oz traces on both layers should carry enough current OR route all non-trace wires (2.5mm) on back side raise signal wire ziptie holes XT-30 FP polarity is wrong"
- note removed: "TODO: current sensing removable current limiting - https://www.powerctc.com/en/node/4564 Errata: JUST FLIP AN ESC UPSIDE DOWN TO FIX TOPOLOGY ISSUES Investigate using traces with vias for high current 10mm 2oz traces on both layers should carry enough current OR route all non-trace wires (2.5mm) on back side raise signal wire ziptie holes XT-30 FP polarity is wrong"
- company: (none) -> Alfredo
- title: (none) -> Spin-Eggman
Changed lines of the file:
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@@
 (kicad_sch (version 20211123) (generator eeschema)
   (paper "A4")
+  (title_block
+    (title "Spin-Eggman")
+    (date "2022-10-20")
+    (rev "V2.0.0")
+    (company "Alfredo")
+  )
   (junction (at 181.61 105.41) (diameter 0) (color 0 0 0 0)
   )
@@
     (effects (font (size 1.27 1.27)) (justify left bottom))
   )
-  (text "TODO:\ncurrent sensing\nremovable current limiting - https://www.powerctc.com/en/node/4564\n\nErrata:\nJUST FLIP AN ESC UPSIDE DOWN TO FIX TOPOLOGY ISSUES\nInvestigate using traces with vias for high current\n10mm 2oz traces on both layers should carry enough current\nOR route all non-trace wires (2.5mm) on back side\nraise signal wire ziptie holes\nXT-30 FP polarity is wrong\n"
+  (text "TODO:\nstartup current limiting - https://www.powerctc.com/en/node/4564\n\nErrata:\nFlip an ESC upside down to fix topology issue\nInvestigate using traces with vias for high current\n10mm 2oz traces on both layers should carry enough current\nOR route all non-trace wires (2.5mm) on back side\nraise signal wire ziptie holes\nXT-30 FP polarity is wrong\n"
     (at 15.24 36.83 0)
     (effects (font (size 1.27 1.27)) (justify left bottom))
