File: spin-sonic/spin-sonic.kicad_pcb (KiCad board)
At the start: 4 copper layers, 66 x 38 mm, 90 parts, among them J1 G-Switch-ST-0322, J2 G-Switch-ST-0322, J4 Conn_01x01, J5 Conn_01x01, J6 Conn_01x01, J64 Conn_01x01_Female, J65 Conn_01x01_Female, J7 Conn_01x01, J8 Conn_01x06, Q11 AO3401A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

Commit message: file cleanup
Other:
- board text added: "SPIN-SONIC V2"
- board text added: "© Alfredo Systems 2022"
- board text removed: "SPIN-TGD-SONIC V2"
- board text removed: "© Jacob Williams 2022"
Changed lines of the file:
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@@
     (effects (font (size 0.8 0.8) (thickness 0.2)) (justify mirror))
   )
-  (gr_text "© Jacob Williams 2022" (at -14.9 0.9) (layer "F.SilkS")
+  (gr_text "© Alfredo Systems 2022" (at -14.566666 0.9) (layer "F.SilkS")
     (effects (font (size 0.8 0.8) (thickness 0.2)))
   )
@@
     (effects (font (size 0.8 0.8) (thickness 0.2)))
   )
-  (gr_text "SPIN-TGD-SONIC V2" (at -15.9 2.3) (layer "F.SilkS")
+  (gr_text "SPIN-SONIC V2" (at -17.5 2.3) (layer "F.SilkS")
     (effects (font (size 0.8 0.8) (thickness 0.2)))
   )
