File: spin-sonic/spin-sonic.kicad_sch (KiCad schematic)
At the start: 53 parts, among them J1 G-Switch-ST-0322, J2 G-Switch-ST-0322, J4 Conn_01x01, J5 Conn_01x01, J6 Conn_01x01, J7 Conn_01x01, J8 Conn_01x06, Q11 AO3401A, Q12 AO3401A, U1 STM32F405RGTx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

Commit message: added image folder and Spin-Sonic PDF
Other:
- title: spin-tgd-control -> Spin-Sonic
Changed lines of the file:
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@@
   (paper "A4")
   (title_block
-    (title "spin-tgd-control")
-    (date "2022-05-12")
+    (title "Spin-Sonic")
+    (date "2022-10-20")
     (rev "V2.0.0")
     (company "Team Alfredo")
